File: Eagle/try1.sch (EAGLE design)
At the start: 7 parts, among them M1 WIRELESS-NRF24L01

Commit message: Just cleaning up and updating the eagle files.
Parts:
- removed 3.3V, A1, D5, GND, RAW: (no value), wirepad:2,54/1,0
- added ESC: (no value), con-lstb:MA03-1
- added H1, H2: MOUNT-PAD-ROUND3.0, holes:MOUNT-PAD-ROUND3.0
- added POTENTIOMETER: (no value), pinhead:PINHD-1X3
Connections:
- removed net IRQ: M1.IRQ, U$2.D2
- removed net N$1: D5.P, U$2.D5
- removed net N$2: A1.P, U$2.A1
- removed net N$3: RAW.P, U$2.RAW
- new net RAW: ESC.2, U$2.RAW
- new net SIG: ESC.1, POTENTIOMETER.1, U$2.A1, U$2.D5
- net GND: now also ESC.3, POTENTIOMETER.3; no longer GND.P, U$2.GND2
- net VCC: now also POTENTIOMETER.2; no longer 3.3V.P, U$2.VCC1
